Commit message: Update SITL to support GPS2 interface

File: models/rotors_description/urdf/component_snippets.xacro (robot description, xacro)
@@ -119,9 +119,10 @@
   </xacro:macro>
   <!-- Macro to add the gps_plugin. -->
-  <xacro:macro name="gps_plugin_macro" params="namespace gps_noise">
+  <xacro:macro name="gps_plugin_macro" params="namespace gps_noise gps_topic">
     <gazebo>
       <plugin name="gps_plugin" filename="libgazebo_gps_plugin.so">
         <robotNamespace>${namespace}</robotNamespace>
         <gpsNoise>${gps_noise}</gpsNoise>
+        <gpsTopic>${gps_topic}</gpsTopic>
       </plugin>
     </gazebo>
@@ -151,5 +152,5 @@
   </xacro:macro>
   <!-- Macro to add the mavlink interface. -->
-  <xacro:macro name="mavlink_interface_macro" params="namespace imu_sub_topic gps_sub_topic mag_sub_topic baro_sub_topic mavlink_addr mavlink_udp_port mavlink_tcp_port serial_enabled serial_device baudrate qgc_addr qgc_udp_port sdk_addr sdk_udp_port hil_mode hil_state_level vehicle_is_tailsitter send_vision_estimation send_odometry enable_lockstep use_tcp">
+  <xacro:macro name="mavlink_interface_macro" params="namespace imu_sub_topic gps_sub_topic gps2_sub_topic mag_sub_topic baro_sub_topic mavlink_addr mavlink_udp_port mavlink_tcp_port serial_enabled serial_device baudrate qgc_addr qgc_udp_port sdk_addr sdk_udp_port hil_mode hil_state_level vehicle_is_tailsitter send_vision_estimation send_odometry enable_lockstep use_tcp">
     <gazebo>
       <plugin name="mavlink_interface" filename="libgazebo_mavlink_interface.so">
@@ -157,4 +158,5 @@
         <imuSubTopic>${imu_sub_topic}</imuSubTopic>
         <gpsSubTopic>${gps_sub_topic}</gpsSubTopic>
+        <gps2SubTopic>${gps2_sub_topic}</gps2SubTopic>
         <magSubTopic>${mag_sub_topic}</magSubTopic>
         <baroSubTopic>${baro_sub_topic}</baroSubTopic>

File: models/rotors_description/urdf/iris_base.xacro (robot description, xacro)
@@ -49,4 +49,12 @@
     namespace="${namespace}"
     gps_noise="true"
+    gps_topic="/gps"
+    >
+  </xacro:gps_plugin_macro>
+  <!-- Instantiate gps2 plugin. -->
+  <xacro:gps_plugin_macro
+    namespace="${namespace}"
+    gps_noise="true"
+    gps_topic="/gps2"
     >
   </xacro:gps_plugin_macro>
@@ -74,4 +82,5 @@
     imu_sub_topic="/imu"
     gps_sub_topic="/gps"
+    gps2_sub_topic="/gps2"
     mag_sub_topic="/mag"
     baro_sub_topic="/baro"

Commit message: Add test gazebo plugin

File: models/rotors_description/urdf/component_snippets.xacro (robot description, xacro)
@@ -592,3 +592,11 @@
     </xacro:imu_plugin_macro>
   </xacro:macro>
+  <xacro:macro name="gazebo_ros_imu_sensor_macro" params="namespace frame_id">
+    <gazebo>
+      <plugin name="gazebo_ros_imu_sensor" filename="libgazebo_ros_imu_sensor.so">
+        <robotNamespace>${namespace}</robotNamespace>
+        <frameName>${frame_id}</frameName>
+      </plugin>
+    </gazebo>
+  </xacro:macro>
 </robot>

File: models/rotors_description/urdf/iris_base.xacro (robot description, xacro)
@@ -191,3 +191,8 @@
     </xacro:bag_plugin_macro>
   </xacro:if>
+  <xacro:gazebo_ros_imu_sensor_macro
+    namespace="${namespace}"
+    frame_id="base_link"
+  >
+  </xacro:gazebo_ros_imu_sensor_macro>
 </robot>

Commit message: Add gps noise params

File: models/rotors_description/urdf/component_snippets.xacro (robot description, xacro)
@@ -119,5 +119,5 @@
   </xacro:macro>
   <!-- Macro to add the gps_plugin. -->
-  <xacro:macro name="gps_plugin_macro" params="namespace gps_noise gps_topic">
+  <xacro:macro name="gps_plugin_macro" params="namespace gps_noise gps_topic gps_corellation_time gps_xy_random_walk gps_z_random_walk gps_xy_noise_density gps_z_noise_density gps_vxy_noise_density gps_vz_noise_density">
     <gazebo>
       <plugin name="gps_plugin" filename="libgazebo_gps_plugin.so">

File: models/rotors_description/urdf/iris_base.xacro (robot description, xacro)
@@ -50,4 +50,11 @@
     gps_noise="true"
     gps_topic="/gps"
+    gps_corellation_time="60.0"
+    gps_xy_random_walk="2.0"
+    gps_z_random_walk="4.0"
+    gps_xy_noise_density="0.0002"
+    gps_z_noise_density="0.0004"
+    gps_vxy_noise_density="0.2"
+    gps_vz_noise_density="0.4"
     >
   </xacro:gps_plugin_macro>

Commit message: Revert files

File: models/rotors_description/urdf/component_snippets.xacro (robot description, xacro)
@@ -119,17 +119,9 @@
   </xacro:macro>
   <!-- Macro to add the gps_plugin. -->
-  <xacro:macro name="gps_plugin_macro" params="namespace gps_noise gps_topic gps_corellation_time gps_xy_random_walk gps_z_random_walk gps_xy_noise_density gps_z_noise_density gps_vxy_noise_density gps_vz_noise_density">
+  <xacro:macro name="gps_plugin_macro" params="namespace gps_noise">
     <gazebo>
       <plugin name="gps_plugin" filename="libgazebo_gps_plugin.so">
         <robotNamespace>${namespace}</robotNamespace>
         <gpsNoise>${gps_noise}</gpsNoise>
-        <gpsTopic>${gps_topic}</gpsTopic>
-        <gpsCorellationTime>${gps_corellation_time}</gpsCorellationTime>
-        <gpsXYRandomWalk>${gps_xy_random_walk}</gpsXYRandomWalk>
-        <gpsZRandomWalk>${gps_z_random_walk}</gpsZRandomWalk>
-        <gpsXYNoiseDensity>${gps_xy_noise_density}</gpsXYNoiseDensity>
-        <gpsZNoiseDensity>${gps_z_noise_density}</gpsZNoiseDensity>
-        <gpsVXYNoiseDensity>${gps_vxy_noise_density}</gpsVXYNoiseDensity>
-        <gpsVZNoiseDensity>${gps_vz_noise_density}</gpsVZNoiseDensity>
       </plugin>
     </gazebo>
@@ -159,5 +151,5 @@
   </xacro:macro>
   <!-- Macro to add the mavlink interface. -->
-  <xacro:macro name="mavlink_interface_macro" params="namespace imu_sub_topic gps_sub_topic gps2_sub_topic mag_sub_topic baro_sub_topic mavlink_addr mavlink_udp_port mavlink_tcp_port serial_enabled serial_device baudrate qgc_addr qgc_udp_port sdk_addr sdk_udp_port hil_mode hil_state_level vehicle_is_tailsitter send_vision_estimation send_odometry enable_lockstep use_tcp">
+  <xacro:macro name="mavlink_interface_macro" params="namespace imu_sub_topic gps_sub_topic mag_sub_topic baro_sub_topic mavlink_addr mavlink_udp_port mavlink_tcp_port serial_enabled serial_device baudrate qgc_addr qgc_udp_port sdk_addr sdk_udp_port hil_mode hil_state_level vehicle_is_tailsitter send_vision_estimation send_odometry enable_lockstep use_tcp">
     <gazebo>
       <plugin name="mavlink_interface" filename="libgazebo_mavlink_interface.so">
@@ -165,5 +157,4 @@
         <imuSubTopic>${imu_sub_topic}</imuSubTopic>
         <gpsSubTopic>${gps_sub_topic}</gpsSubTopic>
-        <gps2SubTopic>${gps2_sub_topic}</gps2SubTopic>
         <magSubTopic>${mag_sub_topic}</magSubTopic>
         <baroSubTopic>${baro_sub_topic}</baroSubTopic>
@@ -592,11 +583,3 @@
     </xacro:imu_plugin_macro>
   </xacro:macro>
-  <xacro:macro name="gazebo_ros_imu_sensor_macro" params="namespace frame_id">
-    <gazebo>
-      <plugin name="gazebo_ros_imu_sensor" filename="libgazebo_ros_imu_sensor.so">
-        <robotNamespace>${namespace}</robotNamespace>
-        <frameName>${frame_id}</frameName>
-      </plugin>
-    </gazebo>
-  </xacro:macro>
 </robot>

File: models/rotors_description/urdf/iris_base.xacro (robot description, xacro)
@@ -49,26 +49,4 @@
     namespace="${namespace}"
     gps_noise="true"
-    gps_topic="/gps"
-    gps_corellation_time="60.0"
-    gps_xy_random_walk="2.0"
-    gps_z_random_walk="4.0"
-    gps_xy_noise_density="0.0002"
-    gps_z_noise_density="0.0004"
-    gps_vxy_noise_density="0.2"
-    gps_vz_noise_density="0.4"
-    >
-  </xacro:gps_plugin_macro>
-  <!-- Instantiate gps2 plugin. -->
-  <xacro:gps_plugin_macro
-    namespace="${namespace}"
-    gps_noise="true"
-    gps_topic="/gps2"
-    gps_corellation_time="60.0"
-    gps_xy_random_walk="0.2"
-    gps_z_random_walk="0.4"
-    gps_xy_noise_density="0.00002"
-    gps_z_noise_density="0.00004"
-    gps_vxy_noise_density="0.02"
-    gps_vz_noise_density="0.04"
     >
   </xacro:gps_plugin_macro>
@@ -96,5 +74,4 @@
     imu_sub_topic="/imu"
     gps_sub_topic="/gps"
-    gps2_sub_topic="/gps2"
     mag_sub_topic="/mag"
     baro_sub_topic="/baro"
@@ -198,8 +175,3 @@
     </xacro:bag_plugin_macro>
   </xacro:if>
-  <xacro:gazebo_ros_imu_sensor_macro
-    namespace="${namespace}"
-    frame_id="base_link"
-  >
-  </xacro:gazebo_ros_imu_sensor_macro>
 </robot>

Commit message: Add RTK helper plugin

File: models/rotors_description/urdf/component_snippets.xacro (robot description, xacro)
@@ -583,3 +583,11 @@
     </xacro:imu_plugin_macro>
   </xacro:macro>
+  <xacro:macro name="gazebo_ros_rtk_helper_plugin_macro" params="namespace body_frame">
+    <gazebo>
+      <plugin name="gazebo_ros_rtk_helper" filename="libgazebo_ros_rtk_helper.so">
+        <robotNamespace>${namespace}</robotNamespace>
+        <bodyFrame>${body_frame}</bodyFrame>
+      </plugin>
+    </gazebo>
+  </xacro:macro>
 </robot>

File: models/rotors_description/urdf/iris_base.xacro (robot description, xacro)
@@ -175,3 +175,8 @@
     </xacro:bag_plugin_macro>
   </xacro:if>
+  <xacro:gazebo_ros_rtk_helper_plugin_macro
+    namespace="${namespace}"
+    body_frame="base_link"
+  >
+  </xacro:gazebo_ros_rtk_helper_plugin_macro>
 </robot>
